Commit message: Small changes in paths

File: agimus_demo_05_pick_and_place/urdf/tless/obj_01.urdf (robot description, URDF)
Before this commit: robot obj_000001, 1 links, 0 joints
Links:
- link base_link: geometry collision mesh filename=package://agimus_demo_05_pick_and_place/urdf/tless/obj_01.o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 scale=1.0 1.0 1.0; visual mesh filename=package://agimus_demo_05_pick_and_place/urdf/tless/obj_01.o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 scale=1.0 1.0 1.0

File: agimus_demo_05_pick_and_place/urdf/tless/obj_21.urdf (robot description, URDF)
Before this commit: robot obj_000021, 1 links, 0 joints
Links:
- link base_link: geometry collision mesh filename=package://agimus_demo_05_pick_and_place/urdf/tless/obj_21.o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 scale=1.0 1.0 1.0; visual mesh filename=package://agimus_demo_05_pick_and_place/urdf/tless/obj_21.o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 scale=1.0 1.0 1.0

File: agimus_demo_05_pick_and_place/urdf/tless/obj_23.urdf (robot description, URDF)
Before this commit: robot obj_000023, 1 links, 0 joints
Links:
- link base_link: geometry collision mesh filename=package://agimus_demo_05_pick_and_place/urdf/tless/obj_23.o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 scale=1.0 1.0 1.0; visual mesh filename=package://agimus_demo_05_pick_and_place/urdf/tless/obj_23.o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 scale=1.0 1.0 1.0

File: agimus_demo_05_pick_and_place/urdf/tless/obj_26.urdf (robot description, URDF)
Before this commit: robot obj_000026, 1 links, 0 joints
Links:
- link base_link: geometry collision mesh filename=package://agimus_demo_05_pick_and_place/urdf/tless/obj_26.o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 scale=1.0 1.0 1.0; visual mesh filename=package://agimus_demo_05_pick_and_place/urdf/tless/obj_26.o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 scale=1.0 1.0 1.0
