Commit message: Merging my and joseph changes, somehow I made a mess...

File: agimus_demo_05_pick_and_place/urdf/franka_hand.xacro (robot description, xacro)
@@ -24,5 +24,5 @@
       <visual>
         <geometry>
-          <mesh filename="package://${description_pkg}/meshes/robot_arms/fer/visual/finger.dae" />
+          <mesh filename="package://${description_pkg}/meshes/robot_ee/franka_hand_white/visual/finger.dae" />
         </geometry>
       </visual>
@@ -63,5 +63,5 @@
         <origin xyz="0 0 0" rpy="0 0 ${pi}" />
         <geometry>
-          <mesh filename="package://${description_pkg}/meshes/robot_arms/fer/visual/finger.dae" />
+          <mesh filename="package://${description_pkg}/meshes/robot_ee/franka_hand_white/visual/finger.dae" />
         </geometry>
       </visual>

Commit message: merged manually PR from joseph (some structure changed meanwhile)

File: agimus_demo_05_pick_and_place/urdf/franka_hand.xacro (robot description, xacro)
@@ -63,5 +63,5 @@
         <origin xyz="0 0 0" rpy="0 0 ${pi}" />
         <geometry>
-          <mesh filename="package://${description_pkg}/meshes/robot_ee/franka_hand_white/visual/finger.dae" />
+          <mesh filename="package://${description_pkg}/meshes/visual/finger.dae" />
         </geometry>
       </visual>

Commit message: Fix URDF files + add option to use SplineGradientBased.

File: agimus_demo_05_pick_and_place/urdf/franka_hand.xacro (robot description, xacro)
@@ -63,5 +63,5 @@
         <origin xyz="0 0 0" rpy="0 0 ${pi}" />
         <geometry>
-          <mesh filename="package://${description_pkg}/meshes/visual/finger.dae" />
+          <mesh filename="package://${description_pkg}/meshes/robot_ee/franka_hand_white/visual/finger.dae" />
         </geometry>
       </visual>

File: agimus_demo_05_pick_and_place/urdf/tless/obj_01.urdf (robot description, URDF)
Before this commit: robot obj_000001, 1 links, 0 joints
Links:
- link base_link: geometry collision mesh filename=package://agimus_demo_05_pick_and_place/urdf/tless/obj_01.o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 scale=0.001 0.001 0.001; visual mesh filename=package://agimus_demo_05_pick_and_place/urdf/tless/obj_01.o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 scale=0.001 0.001 0.001

File: agimus_demo_05_pick_and_place/urdf/tless/obj_21.urdf (robot description, URDF)
Before this commit: robot obj_000021, 1 links, 0 joints
Links:
- link base_link: geometry collision mesh filename=package://agimus_demo_05_pick_and_place/urdf/tless/obj_21.o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 scale=0.001 0.001 0.001; visual mesh filename=package://agimus_demo_05_pick_and_place/urdf/tless/obj_21.o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 scale=0.001 0.001 0.001

File: agimus_demo_05_pick_and_place/urdf/tless/obj_23.urdf (robot description, URDF)
Before this commit: robot obj_000023, 1 links, 0 joints
Links:
- link base_link: geometry collision mesh filename=package://agimus_demo_05_pick_and_place/urdf/tless/obj_23.o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 scale=0.001 0.001 0.001; visual mesh filename=package://agimus_demo_05_pick_and_place/urdf/tless/obj_23.o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 scale=0.001 0.001 0.001

File: agimus_demo_05_pick_and_place/urdf/tless/obj_26.urdf (robot description, URDF)
Before this commit: robot obj_000026, 1 links, 0 joints
Links:
- link base_link: geometry collision mesh filename=package://agimus_demo_05_pick_and_place/urdf/tless/obj_26.o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 scale=0.001 0.001 0.001; visual mesh filename=package://agimus_demo_05_pick_and_place/urdf/tless/obj_26.o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 scale=0.001 0.001 0.001
