Commit message: Remove usage of custom franka xacro files.

File: agimus_demo_05_pick_and_place/urdf/demo.urdf.xacro (robot description, xacro)
@@ -1,10 +1,63 @@
 <?xml version='1.0' encoding='utf-8'?>
 <robot xmlns:xacro="http://www.ros.org/wiki/xacro" name="panda">
-  <xacro:include filename="$(find agimus_demo_05_pick_and_place)/urdf/franka_robot.xacro"/>
+  <xacro:include filename="$(find franka_description)/robots/fer/fer.urdf.xacro">
+    <!-- <xacro:arg name="with_sc" value="True" /> -->
+  </xacro:include>
   <xacro:include filename="$(find agimus_demo_05_pick_and_place)/urdf/support.urdf.xacro"/>
   <xacro:support/>
-  <xacro:franka_robot arm_id="panda"
-                      joint_limits="${xacro.load_yaml('$(find franka_description)/robots/fer/joint_limits.yaml')}">
-  </xacro:franka_robot>
-  <!-- wall behind the table -->
+  <!-- D435 camera -->
+  <xacro:property name="camera_pose_file"
+                  value="$(find agimus_demo_05_pick_and_place)/config/calibrated-params.yaml" />
+  <xacro:property name="camera_pose" value="${load_yaml(camera_pose_file)}"/>
+  <link name="fer_ref_camera_link"/>
+  <joint name="fer_ref_camera_joint" type="fixed">
+    <parent link="fer_hand"/>
+    <child link="fer_ref_camera_link"/>
+    <origin xyz="${camera_pose['camera']['x']}
+                  ${camera_pose['camera']['y']}
+                  ${camera_pose['camera']['z']}"
+      rpy="${camera_pose['camera']['roll']}
+                  ${camera_pose['camera']['pitch']}
+                  ${camera_pose['camera']['yaw']}"/>
+  </joint>
+  <xacro:include filename="$(find realsense2_description)/urdf/_d435.urdf.xacro" />
+  <xacro:sensor_d435 parent="fer_ref_camera_link" name="camera" use_nominal_extrinsics="true">
+    <origin xyz="0 0 0" rpy="0 0 0"/>
+  </xacro:sensor_d435>
+  <!-- camera support -->
+  <link name="fer_camera_support_link">
+    <inertial>
+      <mass value="0.010"/>
+      <origin xyz="0 0 0"/>
+      <inertia ixx="0.001" iyy="0.001" izz="0.001" ixy="0" iyz="0" ixz="0"/>
+    </inertial>
+    <visual>
+      <origin xyz="0.022 0 -0.012" rpy="3.141592653589793 0 -1.5707963267948966"/>
+      <geometry>
+        <mesh filename="package://agimus_demo_05_pick_and_place/urdf/meshes/camera-support.stl" scale="1 1 1"/>
+      </geometry>
+    </visual>
+    <collision>
+      <origin xyz="0.022 0 -0.012" rpy="3.141592653589793 0 -1.5707963267948966"/>
+      <geometry>
+        <mesh filename="package://agimus_demo_05_pick_and_place/urdf/meshes/camera-support.stl" scale="1 1 1"/>
+      </geometry>
+    </collision>
+  </link>
+  <joint name="fer_camera_support_joint" type="fixed">
+    <parent link="fer_hand"/>
+    <child link="fer_camera_support_link"/>
+    <origin xyz="0 0 0" rpy="3.141592653589793 0 0"/>
+  </joint>
+  <xacro:if value="$(arg gazebo)">
+    <xacro:include filename="$(find agimus_demos)/urdf/_d435.gazebo.xacro"/>
+    <xacro:gazebo_d435 camera_name="d435"
+                        reference_link="fer_ref_camera_link"
+                        topics_ns="camera"
+                        depth_optical_frame="camera_depth_optical_frame"
+                        color_optical_frame="camera_color_optical_frame"
+                        infrared1_optical_frame="camera_infrared1_optical_frame"
+                        infrared2_optical_frame="camera_infrared2_optical_frame">
+    </xacro:gazebo_d435>
+  </xacro:if>
 </robot>

File: agimus_demo_05_pick_and_place/urdf/support.urdf.xacro (robot description, xacro)
@@ -157,5 +157,5 @@
         <origin xyz="0.563 -0.1655 .78" rpy="0 0 ${pi}" />
         <parent link="support_link" />
-        <child  link="panda_link0" />
+        <child  link="base" />
       </joint>
       <joint name="wall_joint_1" type="fixed">

Commit message: remove camera from urdf as it is now in franka_description

File: agimus_demo_05_pick_and_place/urdf/demo.urdf.xacro (robot description, xacro)
@@ -6,48 +6,4 @@
   <xacro:include filename="$(find agimus_demo_05_pick_and_place)/urdf/support.urdf.xacro"/>
   <xacro:support/>
-  <!-- D435 camera -->
-  <xacro:property name="camera_pose_file"
-                  value="$(find agimus_demo_05_pick_and_place)/config/calibrated-params.yaml" />
-  <xacro:property name="camera_pose" value="${load_yaml(camera_pose_file)}"/>
-  <link name="fer_ref_camera_link"/>
-  <joint name="fer_ref_camera_joint" type="fixed">
-    <parent link="fer_hand"/>
-    <child link="fer_ref_camera_link"/>
-    <origin xyz="${camera_pose['camera']['x']}
-                  ${camera_pose['camera']['y']}
-                  ${camera_pose['camera']['z']}"
-      rpy="${camera_pose['camera']['roll']}
-                  ${camera_pose['camera']['pitch']}
-                  ${camera_pose['camera']['yaw']}"/>
-  </joint>
-  <xacro:include filename="$(find realsense2_description)/urdf/_d435.urdf.xacro" />
-  <xacro:sensor_d435 parent="fer_ref_camera_link" name="camera" use_nominal_extrinsics="true">
-    <origin xyz="0 0 0" rpy="0 0 0"/>
-  </xacro:sensor_d435>
-  <!-- camera support -->
-  <link name="fer_camera_support_link">
-    <inertial>
-      <mass value="0.010"/>
-      <origin xyz="0 0 0"/>
-      <inertia ixx="0.001" iyy="0.001" izz="0.001" ixy="0" iyz="0" ixz="0"/>
-    </inertial>
-    <visual>
-      <origin xyz="0.022 0 -0.012" rpy="3.141592653589793 0 -1.5707963267948966"/>
-      <geometry>
-        <mesh filename="package://agimus_demo_05_pick_and_place/urdf/meshes/camera-support.stl" scale="1 1 1"/>
-      </geometry>
-    </visual>
-    <collision>
-      <origin xyz="0.022 0 -0.012" rpy="3.141592653589793 0 -1.5707963267948966"/>
-      <geometry>
-        <mesh filename="package://agimus_demo_05_pick_and_place/urdf/meshes/camera-support.stl" scale="1 1 1"/>
-      </geometry>
-    </collision>
-  </link>
-  <joint name="fer_camera_support_joint" type="fixed">
-    <parent link="fer_hand"/>
-    <child link="fer_camera_support_link"/>
-    <origin xyz="0 0 0" rpy="3.141592653589793 0 0"/>
-  </joint>
   <xacro:if value="$(arg gazebo)">
     <xacro:include filename="$(find agimus_demos)/urdf/_d435.gazebo.xacro"/>

Commit message: [demo 5] Clean the URDF files

File: agimus_demo_05_pick_and_place/urdf/demo.urdf.xacro (robot description, xacro)
@@ -6,3 +6,7 @@
   <xacro:include filename="$(find agimus_demo_05_pick_and_place)/urdf/support.urdf.xacro"/>
   <xacro:support/>
+  <joint name="attach_robot_joint" type="fixed">
+    <parent link="robot_attachment_link" />
+    <child link="base" />
+</joint>
 </robot>

File: agimus_demo_05_pick_and_place/urdf/support.urdf.xacro (robot description, xacro)
@@ -154,39 +154,33 @@
       </visual>
     </link>
-    <!-- Gazebo requires a joint to a link called "world" for statically mounted robots -->
-    <link name="world" />
-    <joint name="world_joint" type="fixed">
-      <origin xyz="0 0 0" rpy="0 0 0" />
-      <parent link="world" />
-      <child link="support_link" />
-    </joint>
+    <link name="robot_attachment_link" />
     <joint name="support_joint" type="fixed">
       <origin xyz="0.563 -0.1655 .78" rpy="0 0 ${pi}" />
       <parent link="support_link" />
-      <child link="base" />
+      <child link="robot_attachment_link" />
     </joint>
     <joint name="wall_joint_1" type="fixed">
       <origin xyz="0 1.07 0" />
-      <parent link="world" />
+      <parent link="support_link" />
       <child link="wall_link_1" />
     </joint>
     <joint name="wall_joint_2" type="fixed">
       <origin xyz="1.78 0 0" />
-      <parent link="world" />
+      <parent link="support_link" />
       <child link="wall_link_2" />
     </joint>
     <joint name="wall_joint_3" type="fixed">
       <origin xyz="1.40 0.96 0" />
-      <parent link="world" />
+      <parent link="support_link" />
       <child link="wall_link_3" />
     </joint>
     <joint name="pedestal_joint" type="fixed">
       <origin xyz="1.05 0 0" />
-      <parent link="world" />
+      <parent link="support_link" />
       <child link="pedestal" />
     </joint>
     <joint name="panda1_box_joint" type="fixed">
       <origin xyz="-0.6315 0 1.17" />
-      <parent link="world" />
+      <parent link="support_link" />
       <child link="panda1_box" />
     </joint>
