Commit message: Bypass bug in setRootJointPosition in hpp-manipulation

File: agimus_demo_05_pick_and_place/urdf/small_box.urdf (robot description, URDF)
Before this commit: robot small_box, 1 links, 0 joints
Links:
- added link fake_base_link
Joints:
- added joint fake_joint: type fixed, parent fake_base_link, child base_link

Commit message: Commit changes before vacation, used this for video rec

File: agimus_demo_05_pick_and_place/urdf/small_box.urdf (robot description, URDF)
Before this commit: robot small_box, 2 links, 1 joints
Links:
- link base_link: geometry collision box size=0.001 0.146 0.1; collision box size=0.001 0.146 0.1
