Commit message: update environment

File: agimus_demo_05_pick_and_place/urdf/environment.urdf.xacro (robot description, xacro)
@@ -1,5 +1,12 @@
 <?xml version='1.0' encoding='utf-8'?>
 <robot xmlns:xacro="http://www.ros.org/wiki/xacro" name="environment">
-  <xacro:include filename="$(find agimus_demo_05_pick_and_place)/urdf/support.urdf.xacro"/>
-  <xacro:support/>
+  <xacro:include filename="$(find agimus_demo_05_pick_and_place)/urdf/support.urdf.xacro" />
+  <xacro:support />
+  <joint name="support_to_box" type="fixed">
+    <parent link="support_link" />
+    <child link="big_box_link" />
+    <origin xyz="0.06 -0.2 0.761" />
+  </joint>
+  <xacro:include
+    filename="$(find agimus_demo_05_pick_and_place)/urdf/obstacles.xacro" />
 </robot>

File: agimus_demo_05_pick_and_place/urdf/obstacles.xacro (robot description, xacro)
@@ -1,11 +1,11 @@
 <?xml version='1.0' encoding='utf-8'?>
-<robot xmlns:xacro="http://www.ros.org/wiki/xacro" name="pandas">
+<robot xmlns:xacro="http://www.ros.org/wiki/xacro" name="obstacles">
     <xacro:include filename="$(find franka_description)/robots/common/utils.xacro" />
-    <material name="grey">
-        <color rgba=".5 .5 .5 1" />
+    <material name="red">
+        <color rgba=".9 .1 .1 1" />
     </material>
-    <link name="obstacle1">
+    <link name="big_box_link">
         <inertial>
-            <origin xyz="0.0 0.0 0.0" rpy="0 0 0" />
+            <origin xyz="0 0 0" rpy="0 0 0" />
             <mass value="0.6" />
             <inertia ixx="0.001" ixy="0.0" ixz="0.0"
@@ -18,6 +18,71 @@
                 <box size="0.597 0.397 0.001" />
             </geometry>
-            <color name="grey" />
+            <material name="red" />
         </visual>
+        <collision>
+            <origin xyz="0 0 0.0155" rpy="0 0 0" />
+            <geometry>
+                <box size="0.597 0.397 0.001" />
+            </geometry>
+        </collision>
+        <visual>
+            <origin xyz="0 0.1835 0.12" />
+            <geometry>
+                <box size="0.567 0.001 0.22" />
+            </geometry>
+            <material name="red" />
+        </visual>
+        <collision>
+            <origin xyz="0 0.1835 0.12" />
+            <geometry>
+                <box size="0.567 0.001 0.22" />
+            </geometry>
+        </collision>
+        <visual>
+            <origin xyz="0 -0.1835 0.12" />
+            <geometry>
+                <box size="0.567 0.001 0.22" />
+            </geometry>
+            <material name="red" />
+        </visual>
+        <collision>
+            <origin xyz="0 -0.1835 0.12" />
+            <geometry>
+                <box size="0.567 0.001 0.22" />
+            </geometry>
+        </collision>
+        <visual>
+            <origin xyz="0.2835 0 0.12" />
+            <geometry>
+                <box size="0.001 0.367 0.22" />
+            </geometry>
+            <material name="red" />
+        </visual>
+        <collision>
+            <origin xyz="0.2835 0 0.12" />
+            <geometry>
+                <box size="0.001 0.367 0.22" />
+            </geometry>
+        </collision>
+        <visual>
+            <origin xyz="-0.2835 0 0.12" />
+            <geometry>
+                <box size="0.001 0.367 0.22" />
+            </geometry>
+            <material name="red" />
+        </visual>
+        <collision>
+            <origin xyz="-0.2835 0 0.12" />
+            <geometry>
+                <box size="0.001 0.367 0.22" />
+            </geometry>
+        </collision>
+    </link>
+    <joint name="box_to_obstacle" type="fixed">
+        <parent link="big_box_link" />
+        <child link="obstacle1" />
+        <origin xyz="0.1 0 0.5" rpy="0 0 0 " />
+    </joint>
+    <link name="obstacle1">
         <xacro:collision_capsule xyz="0.535 0 0.43" direction="x" radius="0.1"
             length="0.3" />
