Commit message: improve controller

File: agimus_demo_03_mpc_dummy_traj/urdf/obstacles.xacro (robot description, xacro)
@@ -14,5 +14,5 @@
         </inertial>
         <visual>
-            <origin xyz="0 0 0.0155" rpy="0 0 0" />
+            <origin xyz="0 0 0.0" rpy="0 0 0" />
             <geometry>
                 <box size="0.597 0.397 0.001" />
@@ -20,5 +20,5 @@
             <color name="grey" />
         </visual>
-        <xacro:collision_capsule xyz="0.535 0 0.43" direction="x" radius="0.1"
+        <xacro:collision_capsule xyz="0.43 0.25 0.58" direction="x" radius="0.1"
             length="0.3" />
     </link>
