Commit message: Remove the dependency to frank_description in demo 03_tiago_pro

File: agimus_demo_03_mpc_dummy_traj_tiago_pro/urdf/obstacles.xacro (robot description, xacro)
@@ -1,5 +1,45 @@
 <?xml version='1.0' encoding='utf-8'?>
 <robot xmlns:xacro="http://www.ros.org/wiki/xacro" name="obstacle">
-    <xacro:include filename="$(find franka_description)/robots/common/utils.xacro" />
+    <!-- =========================================================== -->
+    <!-- Add a <collision> tag with a capsule, made from a cylinder  -->
+    <!-- with two spheres at its caps. The capsule will always be    -->
+    <!-- aligned with the axis of 'direction' you pass along.        -->
+    <!--                                                             -->
+    <!-- radius: Radii of both the cylinder and both spheres [m]     -->
+    <!-- length: Length of the cylinder/distance between the centers -->
+    <!--         of the spheres. NOT overall length of capsule!      -->
+    <!-- xyz:    Position of the center of the capsule/cylinder      -->
+    <!-- direction: One of { x, y, z, -x, -y, -z }                   -->
+    <!-- =========================================================== -->
+    <xacro:macro name="collision_capsule" params="radius length xyz:='0 0 0' direction:='z'">
+        <xacro:property name="r" value="${pi/2.0 if 'y' in direction else 0}" />
+        <xacro:property name="p" value="${pi/2.0 if 'x' in direction else 0}" />
+        <xacro:property name="y" value="0" />
+        <xacro:property name="x" value="${xyz.split(' ')[0]}" />
+        <xacro:property name="y" value="${xyz.split(' ')[1]}" />
+        <xacro:property name="z" value="${xyz.split(' ')[2]}" />
+        <!-- Sphere center offsets from center of cylinder -->
+        <xacro:property name="sx" value="${length / 2.0 if 'x' in direction else 0}" />
+        <xacro:property name="sy" value="${length / 2.0 if 'y' in direction else 0}" />
+        <xacro:property name="sz" value="${length / 2.0 if 'z' in direction else 0}" />
+        <collision>
+        <origin xyz="${x} ${y} ${z}" rpy="${r} ${p} ${y}"/>
+        <geometry>
+            <cylinder radius="${radius}" length="${length}" />
+        </geometry>
+        </collision>
+        <collision>
+        <origin xyz="${x+sx} ${y+sy} ${z+sz}" />
+        <geometry>
+            <sphere radius="${radius}" />
+        </geometry>
+        </collision>
+        <collision>
+        <origin xyz="${x-sx} ${y-sy} ${z-sz}" />
+        <geometry>
+            <sphere radius="${radius}" />
+        </geometry>
+        </collision>
+    </xacro:macro>
     <material name="grey">
         <color rgba=".5 .5 .5 1" />
