Commit message: Initial work on manipulation rrt code

File: agimus_demo_06_regrasp/urdf/support.urdf.xacro (robot description, xacro)
@@ -131,4 +131,26 @@
       </collision>
     </link>
+    <link name="foam_block">
+      <inertial>
+        <mass value="1." />
+        <origin xyz="1.05 0.45 0.4625" />
+        <inertia ixx=".01" iyy=".01" izz=".1" ixy="0" ixz="0" iyz="0" />
+      </inertial>
+      <visual>
+        <origin xyz="0 0 0.035" />
+        <geometry>
+          <box size="0.25 0.4 0.07" />
+        </geometry>
+        <material name="transp_blue">
+          <color rgba="0 0.3 0.9 0.5" />
+        </material>
+      </visual>
+      <collision>
+        <origin xyz="0 0 0.035" />
+        <geometry>
+          <box size="0.25 0.4 0.07" />
+        </geometry>
+      </collision>
+    </link>
     <!-- <link name="obj_pedestal">
       <inertial>
@@ -224,9 +246,9 @@
       <child link="pedestal" />
     </joint>
-    <!-- <joint name="obj_pedestal_joint" type="fixed">
+    <joint name="foam_block_joint" type="fixed">
       <origin xyz="0.08 -0.08 0.77" />
       <parent link="support_link" />
-      <child link="obj_pedestal" />
-    </joint> -->
+      <child link="foam_block" />
+    </joint>
     <!-- <joint name="obj_pedestal2_joint" type="fixed">
       <origin xyz="0 0 0.2" />

Commit message: Save changes from robot machine

File: agimus_demo_06_regrasp/urdf/support.urdf.xacro (robot description, xacro)
@@ -11,5 +11,5 @@
         <origin xyz="0 0 0.38" />
         <geometry>
-          <box size="1.703 0.803 0.76" />
+          <box size="1.703 1.803 0.76" />
         </geometry>
         <material name="blue">
@@ -20,5 +20,5 @@
         <origin xyz="0 0 0.38" />
         <geometry>
-          <box size="1.703 0.803 0.76" />
+          <box size="1.703 1.803 0.76" />
         </geometry>
       </collision>
@@ -35,5 +35,5 @@
           </geometry>
         </collision-->
-      <visual>
+      <!-- <visual>
         <origin xyz="0.6385 -0.1655 0.77" />
         <geometry>
@@ -47,5 +47,5 @@
           <box size="0.3 0.3 0.02" />
         </geometry>
-      </collision>
+      </collision> -->
     </link>
     <link name="wall_link_1">
@@ -138,7 +138,7 @@
       </inertial>
       <visual>
-        <origin xyz="0 0 0.035" />
-        <geometry>
-          <box size="0.25 0.4 0.07" />
+        <origin xyz="0 0 0.0225" />
+        <geometry>
+          <box size="0.2 0.4 0.045" />
         </geometry>
         <material name="transp_blue">
@@ -147,7 +147,7 @@
       </visual>
       <collision>
-        <origin xyz="0 0 0.035" />
-        <geometry>
-          <box size="0.25 0.4 0.07" />
+        <origin xyz="0 0 0.0225" />
+        <geometry>
+          <box size="0.2 0.4 0.045" />
         </geometry>
       </collision>
@@ -222,5 +222,5 @@
     <link name="robot_attachment_link" />
     <joint name="support_joint" type="fixed">
-      <origin xyz="0.563 -0.1655 .78" rpy="0 0 ${pi}" />
+      <origin xyz="0.563 -0.1655 .76" rpy="0 0 ${pi}" />
       <parent link="support_link" />
       <child link="robot_attachment_link" />
@@ -247,5 +247,5 @@
     </joint>
     <joint name="foam_block_joint" type="fixed">
-      <origin xyz="0.08 -0.08 0.77" />
+      <origin xyz="0.0 -0.08 0.75" />
       <parent link="support_link" />
       <child link="foam_block" />
