Commit message: Update agimus_demo_06_regrasp/urdf/tless/obj_30.urdf
Co-authored-by: Copilot <175728472+Copilot@users.noreply.github.com>

File: agimus_demo_06_regrasp/urdf/tless/obj_30.urdf (robot description, URDF)
Before this commit: robot obj_000030, 1 links, 0 joints
Links:
- link base_link: geometry collision mesh filename=package://agimus_demo_05_pick_and_place/urdf/tless/obj_30.o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 scale=0.001 0.001 0.001; visual mesh filename=package://agimus_demo_06_regrasp/urdf/tless/obj_30.obj scale=0.001 0.001 0.001
