Commit message: Tune the demo for entering the pylone

File: agimus_demo_07_deburring/environment/pylone.urdf (robot description, URDF)
Before this commit: robot pylone, 1 links, 0 joints
Links:
- added link base_box, mass 5.0; collision box size=0.55 0.52 0.435; visual box size=0.55 0.52 0.435
Joints:
- added joint side_to_pylone: type fixed, parent pylone_link, child base_box, origin xyz=0 0.015 -0.52 rpy=0 0 0.02

File: agimus_demo_07_deburring/urdf/environment.urdf.xacro (robot description, xacro)
@@ -37,5 +37,5 @@
     <visual>
       <geometry>
-        <box size="0.55 0.52 0.532"/>
+        <box size="0.55 0.52 0.435"/>
       </geometry>
       <material name="blue"/>
@@ -43,5 +43,5 @@
     <collision>
       <geometry>
-        <box size="0.55 0.52 0.532"/>
+        <box size="0.55 0.52 0.435"/>
       </geometry>
     </collision>
@@ -68,5 +68,5 @@
     <parent link="base_box"/>
     <child link="pylone_link"/>
-    <origin xyz="0 -0.015 0.55" rpy="0 0 0.02"/>
+    <origin xyz="0 -0.015 0.50" rpy="0 0 0.02"/>
   </joint>
   <xacro:pylone with_sc="$(arg with_sc)" />

File: agimus_demo_07_deburring/urdf/pylone.urdf.xacro (robot description, xacro)
@@ -31,12 +31,18 @@
          <link name="pylone_sc_link">
             <!-- Side edges representing the hole -->
-            <xacro:collision_capsule xyz="0.03 0.1 -0.045" direction="z" radius="0.005" length="0.6" />
-            <xacro:collision_capsule xyz="0.03 -0.1 -0.045" direction="z" radius="0.005" length="0.6" />
+            <xacro:collision_capsule xyz="0.03 0.1 -0.045" direction="z" radius="0.004" length="0.6" />
+            <xacro:collision_capsule xyz="0.03 -0.1 -0.045" direction="z" radius="0.004" length="0.6" />
             <!-- Top and bottom bard representing the hole -->
-            <xacro:collision_capsule xyz="0.03 0.0 ${0.15 - 0.045}" direction="y" radius="0.005" length="0.4" />
-            <xacro:collision_capsule xyz="0.03 0.0 ${-0.15 - 0.045}" direction="y" radius="0.005" length="0.4" />
+            <xacro:collision_capsule xyz="0.03 0.0 ${0.15 - 0.045}" direction="y" radius="0.004" length="0.4" />
+            <xacro:collision_capsule xyz="0.03 0.0 ${-0.15 - 0.045}" direction="y" radius="0.004" length="0.4" />
             <!-- Edges of the pytlone -->
-            <xacro:collision_capsule xyz="0.0 0.205 0.0" direction="z" radius="0.005" length="1.3" />
-            <xacro:collision_capsule xyz="0.0 -0.205 0.0" direction="z" radius="0.005" length="1.3" />
+            <xacro:collision_capsule xyz="0.0 0.205 0.0" direction="z" radius="0.004" length="1.3" />
+            <xacro:collision_capsule xyz="0.0 -0.205 0.0" direction="z" radius="0.004" length="1.3" />
+            <collision>
+               <origin rpy="0 0 0" xyz="0.25 0.2025 0.0" />
+               <geometry>
+                  <box size="0.5 0.005 0.55"/>
+               </geometry>
+            </collision>
          </link>
          <joint name="pylone_sc_link_joint" type="fixed">
