Commit message: [dual_arm] Use shorter bar and make plate borders thiner.

File: agimus_demo_04_dual_arm_tiago_pro/urdf/plate.urdf (robot description, URDF)
Before this commit: robot bordered_plate_model, 5 links, 4 joints
Links:
- link plate_border_back: geometry collision box size=0.01 1.0 0.02; visual box size=0.01 1.0 0.02
- link plate_border_front: geometry collision box size=0.01 1.0 0.02; visual box size=0.01 1.0 0.02
- link plate_border_left: geometry collision box size=1.0 0.01 0.02; visual box size=1.0 0.01 0.02
- link plate_border_right: geometry collision box size=1.0 0.01 0.02; visual box size=1.0 0.01 0.02
Joints:
- joint plate_border_back_joint: origin xyz=-0.49 0 0.025 rpy=0 0 0 -> xyz=-0.495 0 0.025 rpy=0 0 0
- joint plate_border_front_joint: origin xyz=0.49 0 0.025 rpy=0 0 0 -> xyz=0.495 0 0.025 rpy=0 0 0
- joint plate_border_left_joint: origin xyz=0 0.49 0.025 rpy=0 0 0 -> xyz=0 0.495 0.025 rpy=0 0 0
- joint plate_border_right_joint: origin xyz=0 -0.49 0.025 rpy=0 0 0 -> xyz=0 -0.495 0.025 rpy=0 0 0
