Commit message: remove dependency to the demo9 from demo4-tiagopro

File: agimus_demo_04_dual_arm_tiago_pro/urdf/table.urdf (robot description, URDF)
Before this commit: robot table, 1 links, 0 joints
Links:
- link base_link: geometry collision mesh filename=package://agimus_demo_04_dual_arm_tiago_pro/meshes/table.stl scale=0.001 0.001 0.001; visual mesh filename=package://agimus_demo_04_dual_arm_tiago_pro/meshes/table.stl scale=0.001 0.001 0.001
