Commit message: Update env | Finish exposing of params

File: agimus_demo_07_deburring/urdf/pylone.urdf.xacro (robot description, xacro)
@@ -22,4 +22,10 @@
             </geometry>
          </collision>
+         <collision>
+            <origin rpy="1.57 0.0 1.57" xyz="0.0 0.0 -0.265" />
+            <geometry>
+               <box size="0.410 0.0025 0.370" />
+            </geometry>
+         </collision>
          <inertial>
             <origin rpy="0 0 0" xyz="0.0 0.0 0.0" />
@@ -32,8 +38,11 @@
             <!-- Side edges representing the hole -->
             <xacro:collision_capsule xyz="0.03 0.1 -0.045" direction="z" radius="0.004" length="0.6" />
-            <xacro:collision_capsule xyz="0.03 -0.1 -0.045" direction="z" radius="0.004" length="0.6" />
+            <xacro:collision_capsule xyz="0.03 -0.1 -0.045" direction="z" radius="0.004"
+               length="0.6" />
             <!-- Top and bottom bard representing the hole -->
-            <xacro:collision_capsule xyz="0.03 0.0 ${0.15 - 0.045}" direction="y" radius="0.004" length="0.4" />
-            <xacro:collision_capsule xyz="0.03 0.0 ${-0.15 - 0.045}" direction="y" radius="0.004" length="0.4" />
+            <xacro:collision_capsule xyz="0.03 0.0 ${0.15 - 0.045}" direction="y" radius="0.004"
+               length="0.4" />
+            <xacro:collision_capsule xyz="0.03 0.0 ${-0.15 - 0.045}" direction="y" radius="0.004"
+               length="0.4" />
             <!-- Edges of the pytlone -->
             <xacro:collision_capsule xyz="0.0 0.205 0.0" direction="z" radius="0.004" length="1.3" />
@@ -42,5 +51,35 @@
                <origin rpy="0 0 0" xyz="0.25 0.2025 0.0" />
                <geometry>
-                  <box size="0.5 0.005 0.55"/>
+                  <box size="0.5 0.005 0.55" />
+               </geometry>
+            </collision>
+            <collision>
+               <origin rpy="0 0 0" xyz="0.25 -0.2025 0.0" />
+               <geometry>
+                  <box size="0.5 0.005 0.55" />
+               </geometry>
+            </collision>
+            <collision>
+               <origin rpy="0.0 0 1.57" xyz="0.032 0.1525 -0.058" />
+               <geometry>
+                  <box size="0.105 0.0025 0.478" />
+               </geometry>
+            </collision>
+            <collision>
+               <origin rpy="0.0 0 1.57" xyz="0.032 -0.1525 -0.058" />
+               <geometry>
+                  <box size="0.105 0.0025 0.478" />
+               </geometry>
+            </collision>
+            <collision>
+               <origin rpy="0.0 0 1.57" xyz="0.032 0.0 0.14" />
+               <geometry>
+                  <box size="0.410 0.0025 0.075" />
+               </geometry>
+            </collision>
+            <collision>
+               <origin rpy="0.0 0 1.57" xyz="0.032 0.0 -0.23" />
+               <geometry>
+                  <box size="0.410 0.0025 0.075" />
                </geometry>
             </collision>

Commit message: Fix OCP YAML creating | Fix handling of URDF

File: agimus_demo_07_deburring/urdf/pylone.urdf.xacro (robot description, xacro)
@@ -22,10 +22,12 @@
             </geometry>
          </collision>
-         <collision>
-            <origin rpy="1.57 0.0 1.57" xyz="0.0 0.0 -0.265" />
-            <geometry>
-               <box size="0.410 0.0025 0.370" />
-            </geometry>
-         </collision>
+         <xacro:if value="${with_sc}">
+            <collision>
+               <origin rpy="1.57 0.0 1.57" xyz="0.0 0.0 -0.265" />
+               <geometry>
+                  <box size="0.410 0.0025 0.370" />
+               </geometry>
+            </collision>
+         </xacro:if>
          <inertial>
             <origin rpy="0 0 0" xyz="0.0 0.0 0.0" />
