Commit message: migration from hpp6 -> hpp8

File: agimus_demo_10_tiago_pro_bar_manip/urdf/table.urdf (robot description, URDF)
Before this commit: robot table, 1 links, 0 joints
Links:
- link table_link: geometry collision mesh filename=package://agimus_demo_10_tiago_pro_bar_manip/meshes/table.s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 scale=0.001 0.001 0.001; visual mesh filename=package://agimus_demo_10_tiago_pro_bar_manip/meshes/table.s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 scale=0.001 0.001 0.001
