Commit message: add bar in gazebo + base odom

File: agimus_demo_10_tiago_pro_bar_manip/urdf/environment.urdf.xacro (robot description, xacro)
@@ -1,15 +1,9 @@
 <?xml version="1.0"?>
-<robot name="environment" xmlns:xacro="http://www.ros.org/wiki/xacro">
+<robot name="environment_static" xmlns:xacro="http://www.ros.org/wiki/xacro">
+  <xacro:include filename="$(find agimus_demo_10_tiago_pro_bar_manip)/urdf/macro/ground_macro.urdf.xacro"/>
+  <xacro:include filename="$(find agimus_demo_10_tiago_pro_bar_manip)/urdf/macro/table_macro.urdf.xacro"/>
+  <xacro:include filename="$(find agimus_demo_10_tiago_pro_bar_manip)/urdf/macro/plate_macro.urdf.xacro"/>
+  <xacro:include filename="$(find agimus_demo_10_tiago_pro_bar_manip)/urdf/macro/support_macro.urdf.xacro"/>
   <link name="world"/>
-  <link name="odom"/>
-  <xacro:include filename="$(find agimus_demo_10_tiago_pro_bar_manip)/urdf/ground.urdf.xacro"/>
-  <xacro:include filename="$(find agimus_demo_10_tiago_pro_bar_manip)/urdf/plate.urdf.xacro"/>
-  <xacro:include filename="$(find agimus_demo_10_tiago_pro_bar_manip)/urdf/reinforcement_bar.urdf.xacro"/>
-  <xacro:include filename="$(find agimus_demo_10_tiago_pro_bar_manip)/urdf/table.urdf.xacro"/>
- <joint name="world_odom" type="fixed">
-    <parent link="world"/>
-    <child link="odom"/>
-    <origin xyz="0 0 0" rpy="0 0 0"/>
-  </joint>
   <xacro:ground/>
   <joint name="ground_world_joint" type="fixed">
@@ -19,22 +13,25 @@
   </joint>
   <xacro:table/>
-  <joint name="table_world_joint" type="floating">
-    <parent link="ground_link"/>
+  <joint name="table_world_joint" type="fixed">
+    <parent link="world"/>
     <child link="table_link"/>
-    <origin xyz="0 0 0" rpy="0 0 0"/>
+    <origin xyz="2.9 0 0" rpy="0 0 3.14"/>
   </joint>
   <xacro:bordered_plate name="plate">
     <origin xyz="0 0 0" rpy="0 0 0"/>
   </xacro:bordered_plate>
-  <joint name="plate_world_joint" type="floating">
-    <parent link="ground_link"/>
+  <joint name="plate_world_joint" type="fixed">
+    <parent link="world"/>
     <child link="plate_base_link"/>
-    <origin xyz="0 0 0" rpy="0 0 0"/>
+    <origin xyz="2.3 0 0.66" rpy="0 0 0"/>
   </joint>
-  <xacro:reinforcement_bar/>
-  <joint name="bar_world_joint" type="floating">
-    <parent link="ground_link"/>
-    <child link="bar_base_link"/>
-    <origin xyz="0 0 0" rpy="0 0 0"/>
+  <xacro:support_bar spacing="0.95"/>
+  <joint name="support_world_joint" type="fixed">
+    <parent link="table_link"/>
+    <child link="support_base_link"/>
+    <origin xyz="1.32 0 0.7" rpy="0 0 ${pi/2}"/>
   </joint>
+  <gazebo>
+    <static>true</static>
+  </gazebo>
 </robot>

File: agimus_demo_10_tiago_pro_bar_manip/urdf/macro/plate_macro.urdf.xacro (robot description, xacro)
@@ -8,4 +8,5 @@
   <xacro:property name="plate_width"  value="${setup_file['plate']['width']}"  /> <!-- Dimension sur l'axe Y -->
   <xacro:property name="plate_height" value="${setup_file['plate']['height']}" /> <!-- Épaisseur de la plaque -->
+  <xacro:property name="plate_mass" value="${setup_file['plate']['mass']}"/>
   <xacro:property name="border_height"    value="${setup_file['plate']['border_height']}" />    <!-- Hauteur des bordures -->
   <xacro:property name="border_thickness" value="${setup_file['plate']['border_thickness']}" /> <!-- Épaisseur des bordures -->
@@ -52,4 +53,12 @@
     <!-- Le maillon de base (la surface de la plaque) -->
     <link name="${name}_base_link">
+      <inertial>
+        <mass value="${plate_mass}"/>
+        <inertia
+          ixx="${plate_mass/12.0 * (plate_width*plate_width + plate_height*plate_height)}"
+          iyy="${plate_mass/12.0 * (plate_length*plate_length + plate_height*plate_height)}"
+          izz="${plate_mass/12.0 * (plate_length*plate_length + plate_width*plate_width)}"
+          ixy="0" ixz="0" iyz="0"/>
+      </inertial>
       <visual>
         <geometry><box size="${plate_length} ${plate_width} ${plate_height}"/></geometry>

File: agimus_demo_10_tiago_pro_bar_manip/urdf/macro/reinforcement_bar_macro.urdf.xacro (robot description, xacro)
@@ -2,5 +2,13 @@
 <robot xmlns:xacro="http://www.ros.org/wiki/xacro">
   <xacro:macro name="reinforcement_bar" params="prefix:=''">
+    <material name="Light-Grey">
+      <color rgba="0.8 0.8 0.8 1.0"/>
+    </material>
     <link name="${prefix}bar_base_link">
+      <inertial>
+        <origin xyz="0.025 0 0"/>
+        <mass value="2.5"/>
+        <inertia ixx="0.02" ixy="0" ixz="0" iyy="0.05" iyz="0" izz="0.04"/>
+      </inertial>
       <collision>
         <origin xyz="0 0 -0.48"/>
@@ -16,4 +24,5 @@
                 scale="0.001 0.001 0.001"/>
         </geometry>
+        <material name="Light-Grey"/>
       </visual>
     </link>

File: agimus_demo_10_tiago_pro_bar_manip/urdf/macro/table_macro.urdf.xacro (robot description, xacro)
@@ -2,5 +2,13 @@
 <robot xmlns:xacro="http://www.ros.org/wiki/xacro">
   <xacro:macro name="table" params="prefix:=''">
+    <material name="Blue">
+      <color rgba="0.0 0.05 0.4 1.0"/>
+    </material>
     <link name="${prefix}table_link">
+      <inertial>
+        <origin xyz="0 0 0"/>
+        <mass value="25.5"/>
+        <inertia ixx="0.02" ixy="0" ixz="0" iyy="0.05" iyz="0" izz="0.04"/>
+      </inertial>
       <visual>
         <origin rpy="0 0 0" xyz="0.6 0 0.585"/>

File: agimus_demo_10_tiago_pro_bar_manip/urdf/standalone/ground.urdf.xacro (robot description, xacro)
@@ -1,5 +1,5 @@
 <?xml version="1.0"?>
 <robot name="ground" xmlns:xacro="http://www.ros.org/wiki/xacro">
-  <xacro:include filename="$(find agimus_demo_10_tiago_pro_bar_manip)/urdf/ground.urdf.xacro"/>
+  <xacro:include filename="$(find agimus_demo_10_tiago_pro_bar_manip)/urdf/macro/ground_macro.urdf.xacro"/>
   <xacro:ground prefix=""/>
 </robot>

File: agimus_demo_10_tiago_pro_bar_manip/urdf/standalone/plate.urdf.xacro (robot description, xacro)
@@ -1,5 +1,5 @@
 <?xml version="1.0"?>
 <robot name="plate" xmlns:xacro="http://www.ros.org/wiki/xacro">
-  <xacro:include filename="$(find agimus_demo_10_tiago_pro_bar_manip)/urdf/plate.urdf.xacro"/>
+  <xacro:include filename="$(find agimus_demo_10_tiago_pro_bar_manip)/urdf/macro/plate_macro.urdf.xacro"/>
   <xacro:bordered_plate name="plate">
     <origin xyz="0 0 0" rpy="0 0 0"/>

File: agimus_demo_10_tiago_pro_bar_manip/urdf/standalone/reinforcement_bar.urdf.xacro (robot description, xacro)
@@ -1,5 +1,16 @@
 <?xml version="1.0"?>
 <robot name="reinforcement_bar" xmlns:xacro="http://www.ros.org/wiki/xacro">
-  <xacro:include filename="$(find agimus_demo_10_tiago_pro_bar_manip)/urdf/reinforcement_bar.urdf.xacro"/>
+  <!-- 1. Ton object géométrique et physique -->
+  <xacro:include filename="$(find agimus_demo_10_tiago_pro_bar_manip)/urdf/macro/reinforcement_bar_macro.urdf.xacro"/>
   <xacro:reinforcement_bar prefix=""/>
+  <!-- 2. Le plugin Gazebo indispensable pour faire le point avec /tf -->
+  <gazebo>
+    <plugin filename="libgz-sim-pose-publisher-system.so" name="gz::sim::systems::PosePublisher">
+      <publish_link_pose>true</publish_link_pose>
+      <publish_model_pose>true</publish_model_pose>
+      <publish_nested_model_pose>true</publish_nested_model_pose>
+      <use_pose_vector_msg>true</use_pose_vector_msg>
+      <update_frequency>50</update_frequency>
+    </plugin>
+  </gazebo>
 </robot>

File: agimus_demo_10_tiago_pro_bar_manip/urdf/standalone/table.urdf.xacro (robot description, xacro)
@@ -1,5 +1,19 @@
+<!-- <?xml version="1.0"?>
+<robot name="table" xmlns:xacro="http://www.ros.org/wiki/xacro">
+  <xacro:include filename="$(find agimus_demo_10_tiago_pro_bar_manip)/urdf/macro/table_macro.urdf.xacro"/>
+  <xacro:table prefix=""/>
+</robot> -->
 <?xml version="1.0"?>
-<robot name="table" xmlns:xacro="http://www.ros.org/wiki/xacro">
-  <xacro:include filename="$(find agimus_demo_10_tiago_pro_bar_manip)/urdf/table.urdf.xacro"/>
+<robot xmlns:xacro="http://www.ros.org/wiki/xacro" name="table">
+  <xacro:include filename="$(find agimus_demo_10_tiago_pro_bar_manip)/urdf/macro/table_macro.xacro"/>
+  <link name="world"/>
   <xacro:table prefix=""/>
+  <joint name="world_to_table" type="fixed">
+    <parent link="world"/>
+    <child link="table_link"/>
+    <origin xyz="2. 0 0" rpy="0 0 0"/>
+  </joint>
+  <gazebo>
+    <static>true</static>
+  </gazebo>
 </robot>

Commit message: Add sim option into launch + cancel exec

File: agimus_demo_10_tiago_pro_bar_manip/urdf/environment.urdf.xacro (robot description, xacro)
@@ -16,5 +16,5 @@
     <parent link="world"/>
     <child link="table_link"/>
-    <origin xyz="2.9 0 0" rpy="0 0 3.14"/>
+    <origin xyz="2.3 0 0.74" rpy="0 0 3.14"/>
   </joint>
   <xacro:bordered_plate name="plate">
@@ -22,7 +22,7 @@
   </xacro:bordered_plate>
   <joint name="plate_world_joint" type="fixed">
-    <parent link="world"/>
+    <parent link="table_link"/>
     <child link="plate_base_link"/>
-    <origin xyz="2.3 0 0.66" rpy="0 0 0"/>
+    <origin xyz="-0.2 0 0" rpy="0 0 0"/>
   </joint>
   <xacro:support_bar spacing="0.95"/>
@@ -30,5 +30,5 @@
     <parent link="table_link"/>
     <child link="support_base_link"/>
-    <origin xyz="1.32 0 0.7" rpy="0 0 ${pi/2}"/>
+    <origin xyz="0.60 0 0" rpy="0 0 ${pi/2}"/>
   </joint>
   <gazebo>

File: agimus_demo_10_tiago_pro_bar_manip/urdf/macro/plate_macro.urdf.xacro (robot description, xacro)
@@ -60,11 +60,18 @@
           izz="${plate_mass/12.0 * (plate_length*plate_length + plate_width*plate_width)}"
           ixy="0" ixz="0" iyz="0"/>
+        <origin xyz="0 0 ${plate_height/2}" rpy="0 0 0"/>
       </inertial>
       <visual>
-        <geometry><box size="${plate_length} ${plate_width} ${plate_height}"/></geometry>
+        <geometry>
+          <box size="${plate_length} ${plate_width} ${plate_height}"/>
+        </geometry>
         <material name="grey"/>
+        <origin xyz="0 0 ${plate_height/2}" rpy="0 0 0"/>
       </visual>
       <collision>
-        <geometry><box size="${plate_length} ${plate_width} ${plate_height}"/></geometry>
+        <geometry>
+          <box size="${plate_length} ${plate_width} ${plate_height}"/>
+        </geometry>
+        <origin xyz="0 0 ${plate_height/2}" rpy="0 0 0"/>
       </collision>
     </link>
@@ -72,21 +79,21 @@
     <!-- Bordure Avant (+X) -->
     <xacro:single_border name="${name}_border_front" parent_link="${name}_base_link"
-                         size_x="${border_thickness}" size_y="${plate_width}" size_z="${border_height}">
-      <origin xyz="${plate_length/2 - border_thickness/2} 0 ${border_height/2 + plate_height/2}" rpy="0 0 0"/>
+                        size_x="${border_thickness}" size_y="${plate_width}" size_z="${border_height}">
+      <origin xyz="${plate_length/2 - border_thickness/2} 0 ${plate_height + border_height/2}" rpy="0 0 0"/>
     </xacro:single_border>
     <!-- Bordure Arrière (-X) -->
     <xacro:single_border name="${name}_border_back" parent_link="${name}_base_link"
-                         size_x="${border_thickness}" size_y="${plate_width}" size_z="${border_height}">
-      <origin xyz="-${plate_length/2 - border_thickness/2} 0 ${border_height/2 + plate_height/2}" rpy="0 0 0"/>
+                        size_x="${border_thickness}" size_y="${plate_width}" size_z="${border_height}">
+      <origin xyz="-${plate_length/2 - border_thickness/2} 0 ${plate_height + border_height/2}" rpy="0 0 0"/>
     </xacro:single_border>
     <!-- Bordure Gauche (+Y) -->
     <xacro:single_border name="${name}_border_left" parent_link="${name}_base_link"
-                         size_x="${plate_length}" size_y="${border_thickness}" size_z="${border_height}">
-      <origin xyz="0 ${plate_width/2 - border_thickness/2} ${border_height/2 + plate_height/2}" rpy="0 0 0"/>
+                        size_x="${plate_length}" size_y="${border_thickness}" size_z="${border_height}">
+      <origin xyz="0 ${plate_width/2 - border_thickness/2} ${plate_height + border_height/2}" rpy="0 0 0"/>
     </xacro:single_border>
     <!-- Bordure Droite (-Y) -->
     <xacro:single_border name="${name}_border_right" parent_link="${name}_base_link"
-                         size_x="${plate_length}" size_y="${border_thickness}" size_z="${border_height}">
-      <origin xyz="0 -${plate_width/2 - border_thickness/2} ${border_height/2 + plate_height/2}" rpy="0 0 0"/>
+                        size_x="${plate_length}" size_y="${border_thickness}" size_z="${border_height}">
+      <origin xyz="0 -${plate_width/2 - border_thickness/2} ${plate_height + border_height/2}" rpy="0 0 0"/>
     </xacro:single_border>
   </xacro:macro>

File: agimus_demo_10_tiago_pro_bar_manip/urdf/macro/table_macro.urdf.xacro (robot description, xacro)
@@ -3,5 +3,5 @@
   <xacro:macro name="table" params="prefix:=''">
     <material name="Blue">
-      <color rgba="0.0 0.05 0.4 1.0"/>
+      <color rgba="0.0 0.0 0.4 1.0"/>
     </material>
     <link name="${prefix}table_link">
@@ -9,17 +9,29 @@
         <origin xyz="0 0 0"/>
         <mass value="25.5"/>
-        <inertia ixx="0.02" ixy="0" ixz="0" iyy="0.05" iyz="0" izz="0.04"/>
+        <inertia ixx="0.02" ixy="0" ixz="0"
+                 iyy="0.05" iyz="0" izz="0.04"/>
       </inertial>
       <visual>
-        <origin rpy="0 0 0" xyz="0.6 0 0.585"/>
+        <origin rpy="0 0 0" xyz="0.35 0 0"/>
         <geometry>
-          <mesh filename="package://agimus_demo_10_tiago_pro_bar_manip/meshes/table.stl" scale="0.001 0.001 0.001"/>
+          <mesh
+            filename="package://agimus_demo_10_tiago_pro_bar_manip/meshes/table.stl"
+            scale="0.001 0.001 0.001"/>
+        </geometry>
+        <material name="Blue"/>
+      </visual>
+      <visual>
+        <origin rpy="0 0 0" xyz="-0.35 0 0"/>
+        <geometry>
+          <mesh
+            filename="package://agimus_demo_10_tiago_pro_bar_manip/meshes/table.stl"
+            scale="0.001 0.001 0.001"/>
         </geometry>
         <material name="Blue"/>
       </visual>
       <collision>
-        <origin rpy="0 0 0" xyz="0.6 0 0.585"/>
+        <origin rpy="0 0 0" xyz="0 0 -0.37"/>
         <geometry>
-          <mesh filename="package://agimus_demo_10_tiago_pro_bar_manip/meshes/table.stl" scale="0.001 0.001 0.001"/>
+          <box size="1.4 1.4 0.74"/>
         </geometry>
       </collision>

File: agimus_demo_10_tiago_pro_bar_manip/urdf/standalone/plate.urdf (robot description, URDF)
Before this commit: robot plate, 5 links, 4 joints
Links:
- link plate_base_link: mass None -> 4.0
Joints:
- joint plate_border_back_joint: origin xyz=-0.49 0 0.025 rpy=0 0 0 -> xyz=-0.49 0 0.04 rpy=0 0 0
- joint plate_border_front_joint: origin xyz=0.49 0 0.025 rpy=0 0 0 -> xyz=0.49 0 0.04 rpy=0 0 0
- joint plate_border_left_joint: origin xyz=0 0.49 0.025 rpy=0 0 0 -> xyz=0 0.49 0.04 rpy=0 0 0
- joint plate_border_right_joint: origin xyz=0 -0.49 0.025 rpy=0 0 0 -> xyz=0 -0.49 0.04 rpy=0 0 0

File: agimus_demo_10_tiago_pro_bar_manip/urdf/standalone/table.urdf (robot description, URDF)
Before this commit: robot table, 1 links, 0 joints
Links:
- link table_link: mass None -> 25.5; geometry collision box size=1.4 1.4 0.74; visual mesh filename=package://agimus_demo_10_tiago_pro_bar_manip/meshes/table.s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 scale=0.001 0.001 0.001

File: agimus_demo_10_tiago_pro_bar_manip/urdf/standalone/table.urdf.xacro (robot description, xacro)
@@ -1,19 +1,5 @@
-<!-- <?xml version="1.0"?>
+<?xml version="1.0"?>
 <robot name="table" xmlns:xacro="http://www.ros.org/wiki/xacro">
   <xacro:include filename="$(find agimus_demo_10_tiago_pro_bar_manip)/urdf/macro/table_macro.urdf.xacro"/>
   <xacro:table prefix=""/>
-</robot> -->
-<?xml version="1.0"?>
-<robot xmlns:xacro="http://www.ros.org/wiki/xacro" name="table">
-  <xacro:include filename="$(find agimus_demo_10_tiago_pro_bar_manip)/urdf/macro/table_macro.xacro"/>
-  <link name="world"/>
-  <xacro:table prefix=""/>
-  <joint name="world_to_table" type="fixed">
-    <parent link="world"/>
-    <child link="table_link"/>
-    <origin xyz="2. 0 0" rpy="0 0 0"/>
-  </joint>
-  <gazebo>
-    <static>true</static>
-  </gazebo>
 </robot>
