Commit message: Add ground into hpp planning

File: agimus_demo_10_tiago_pro_bar_manip/urdf/standalone/plate.urdf (robot description, URDF)
Before this commit: robot bordered_plate_model, 6 links, 5 joints
Links:
- removed link plate_bottom_link
- link plate_base_link: geometry collision box size=1.0 1.0 0.03; visual box size=1.0 1.0 0.03
- link plate_border_back: geometry collision box size=0.02 1.0 0.02; visual box size=0.02 1.0 0.02
- link plate_border_front: geometry collision box size=0.02 1.0 0.02; visual box size=0.02 1.0 0.02
- link plate_border_left: geometry collision box size=1.0 0.02 0.02; visual box size=1.0 0.02 0.02
- link plate_border_right: geometry collision box size=1.0 0.02 0.02; visual box size=1.0 0.02 0.02
Joints:
- removed joint plate_origin_joint
- joint plate_border_back_joint: origin xyz=-0.495 0 0.025 rpy=0 0 0 -> xyz=-0.49 0 0.025 rpy=0 0 0; parent plate_bottom_link -> plate_base_link
- joint plate_border_front_joint: origin xyz=0.495 0 0.025 rpy=0 0 0 -> xyz=0.49 0 0.025 rpy=0 0 0; parent plate_bottom_link -> plate_base_link
- joint plate_border_left_joint: origin xyz=0 0.495 0.025 rpy=0 0 0 -> xyz=0 0.49 0.025 rpy=0 0 0; parent plate_bottom_link -> plate_base_link
- joint plate_border_right_joint: origin xyz=0 0 0 rpy=0 0 0 -> xyz=0 -0.49 0.025 rpy=0 0 0; parent plate_bottom_link -> plate_base_link
